Commit message: Commit improved versions

File: examples/models/twoLinks/model.urdf (robot description, URDF)
Before this commit: robot twoLinks, 5 links, 4 joints
Links:
- link link1: geometry collision box size=0.1 0.1 0.90; visual box size=0.1 0.1 0.90
- link link2: geometry collision cylinder length=0.85 radius=0.05; visual cylinder length=0.85 radius=0.05
Joints:
- joint joint1: origin xyz=0 0 1 rpy=0 -0 0 -> xyz=0 0 0 rpy=0 -0 0
- joint joint2: origin xyz=0 0 1 rpy=0 -0 0 -> xyz=0 0 0 rpy=0 -0 0
- joint joint_end_effector: origin xyz=0 0 0 rpy=0 0 0 -> xyz=0 0 1 rpy=0 0 0
- joint middle_link_joint: origin xyz=0 0 0 rpy=0 0 0 -> xyz=0 0 1 rpy=0 0 0
